File: hardware/pilyzer-afe/kicad/channel-2.kicad_sch (KiCad schematic)
At the start: 20 parts, among them J2 BNC, J4 Input header, U1 TLV9064IDR, U2 TS5A23159DGSR

Commit message: Replace the passive RC pair with a Sallen-Key and drop the BNCs
A third channel divides the converter three ways instead of two, so
Nyquist fell from 124 to 82 kHz and the old passband reached past it:
between 82 kHz and roughly 250 kHz a signal was neither rejected by the
filter nor resolved by the converter, and folded back looking real.

Each channel now ends in a unity-gain Sallen-Key on U4 — R 2.67k, C1
2.2n, C2 1n to VMID — giving fc 40.2 kHz and Q 0.742, so 12.5 dB down at
three-channel Nyquist instead of nearly nothing. The shunt returns to
VMID rather than ground to keep the mid-rail bias ratiometric. R is a
value the board already used and the amplifier is a second TLV9064, so
the whole filter adds one part type to an order.

The BNC footprints are gone; inputs are the 2-pin headers. ERC is clean
and check_kicad.py covers the new topology.

Co-Authored-By: Claude Opus 5 <noreply@anthropic.com>
Parts:
- removed J2: BNC, PiLyzer:BNC_Amphenol_031-6575_Horizontal, symbol PiLyzer:Connector_Conn_Coaxial
- added C22: 2.2n C0G, PiLyzer:C_0603_1608Metric, symbol PiLyzer:Device_C
- added R45: 1k 1%, PiLyzer:R_0805_2012Metric, symbol PiLyzer:Device_R
- added U4: TLV9064IDR, PiLyzer:SOIC-14_3.9x8.7mm_P1.27mm, symbol PiLyzer:Amplifier_Operational_TLV9064
- R13, R14: value 1k 1% -> 2.67k 1%
Connections:
- net CH2_ADC: now also R45.2; no longer R14.2
- net GND: no longer C10.2
- net VMID: now also C10.2
- net CH2_RC1 renamed CH2_SK
- net CH2_SK: now also C22.1; no longer C10.1
- new net CH2_FILT: C22.2, R45.1, U4.6 (-), U4.7
- new net CH2_SKIN: C10.1, R14.2, U4.5 (+)
Other:
- note added: "ANTI-ALIAS FILTER unity-gain Sallen-Key, fc 40.2 kHz, Q 0.742 (C shunt returns to VMID)"
- note added: "Signal flow: input → compensated divider → gain stage → Sallen-Key 40.2 kHz → ADC"
- note added: "U1/U2/U3/U4 supply units and the VMID buffer are on sheet 1. GND includes Pico AGND."
- note removed: "Signal flow: input → compensated divider → amplifier → two RC sections → ADC"
- note removed: "U1/U2 supply units and VMID buffer are on sheet 1. GND includes Pico AGND."
