File: Pico2/hardware/pilyzer-afe/kicad/channel-3.kicad_sch (KiCad schematic)
At the start: 22 parts, among them J10 Input header, U1 TLV9064IDR, U3 TS5A23159DGSR, U4 TLV9064IDR

Commit message: Widen the compensation window, and give Lite a fixed capacitor to aim at
The divider is flat when C_top = C_node / 14.96, and C_node is C4 plus whatever
the layout adds. With C1 at 6.8 pF and TC1 at 0.5–3 pF the adjustable window was
7.3 to 9.8 pF, which is a node stray of 27 to 65 pF — high for a board this
small. Below 27 pF the trimmer bottoms out over-compensated with nowhere left to
go, and the board cannot be trimmed flat at all.

C1 is 5.6 pF now, which puts the window at 6.1 to 8.6 pF and a stray of 9 to
47 pF, straddling what a node with an amplifier input, a clamp, a trimmer body
and a test point on it plausibly comes to.

Measurement would not have caught this. A breadboard's stray is larger than a
PCB's, so it pushes the answer up into the window and trims happily from a board
that could not — the failure would have appeared for the first time on the
fabricated article. So the window is settled by arithmetic beforehand instead.

For Lite the same relation gives a way to drop the trimmer, which is a cost on a
teaching board and something for a student to turn. The larger C4 is, the
smaller a fraction of C_node the unknown stray becomes: at 220 pF a 10 pF error
is 4.2% rather than 9.8%, for an input capacitance of 16 pF against a bench
scope's usual 10 to 20. So Lite takes C4 220 pF and a fixed part near 16 pF,
with the number itself coming from the first boards rather than from the table.

Schematic values changed for C1, C8 and C16 on all three channel sheets. ERC
regenerated: 0 errors, 0 warnings. The netlist check still passes.

Co-Authored-By: Claude Opus 5 <noreply@anthropic.com>
Parts:
- C16: value 6.8p C0G -> 5.6p C0G
