File: Pico2/hardware/pilyzer-afe/kicad/pilyzer-afe.kicad_sch (KiCad schematic)
At the start: 36 parts, among them J5 Logic D0–D7 + GND, J6 Pico 2 socket, J7 Pico 2 socket, U1 TLV9064IDR, U2 TS5A23159DGSR, U3 TS5A23159DGSR, U4 TLV9064IDR

Commit message: Move the rev A range and calibration nets to where the firmware looks
Firmware 1.11 took the range controls down to GPIO4/5/6 so the generator
could have GPIO16-19 on every board, and 1.12 put the square wave on
GPIO22. The schematic still drew the old map, which check_kicad.py has
been reporting ever since; this is the redraw it was asking for.

RANGE_CH1/2/3 move from J7.20/19/17 to J6.6/7/9, and CAL_GPIO20 on J7.15
becomes CAL_GPIO22 on J7.12. Each was a 7.62 mm stub to a global label,
so the nets themselves are unchanged — only which pad they land on. The
no-connect flags swap with them: off the three J6 pads that are now
driven and the J7 pad that now carries the square wave, onto the four
J7 pads the moves vacated.

Verified with the tools rather than by eye: check_kicad.py passes its 54
net groups against the netlist KiCad generates, and ERC is back to 0
errors and 0 warnings from the 8 the first attempt caused — it was ERC
that caught the no-connect flags I had left behind.

The channel previews change too, and not because of this: they were
exported before C1 became 5.6 pF and still drew 6.8 pF. Regenerating all
four brings them level with the schematic and the BOM.

Co-Authored-By: Claude Opus 5 <noreply@anthropic.com>
Connections:
- net RANGE_CH1: now also J6.6 (Pin_6); no longer J7.20 (Pin_20)
- net RANGE_CH2: now also J6.7 (Pin_7); no longer J7.19 (Pin_19)
- net RANGE_CH3: now also J6.9 (Pin_9); no longer J7.17 (Pin_17)
- net CAL_GPIO22: now reaches J7.12 (Pin_12)
- net CAL_GPIO22: now also R35.1
- net CAL_GPIO20: no longer names the net of J7.15 (Pin_15)
- net CAL_GPIO20: no longer R35.1
Other:
- note added: "ADC GPIO26–28; logic GPIO8–15; range GPIO4–6; test GPIO22; generator GPIO16–19."
- note removed: "Firmware 1.5: ADC GPIO26–28; logic GPIO8–15; range GPIO16–18; test GPIO20."
Changed lines of the file:
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@@
 		)
 	)
-	(text "Firmware 1.5: ADC GPIO26–28; logic GPIO8–15; range GPIO16–18; test GPIO20."
+	(text "ADC GPIO26–28; logic GPIO8–15; range GPIO4–6; test GPIO22; generator GPIO16–19."
 		(exclude_from_sim no)
 		(at 12.7 142.24 0)
@@
 	)
 	(no_connect
-		(at 43.18 77.47)
+		(at 114.3 97.79)
 	)
 	(no_connect
@@
 	)
 	(no_connect
-		(at 43.18 72.39)
+		(at 114.3 102.87)
 	)
 	(no_connect
@@
 	)
 	(no_connect
-		(at 43.18 69.85)
+		(at 114.3 105.41)
 	)
 	(no_connect
-		(at 114.3 85.09)
+		(at 114.3 92.71)
 	)
 	(no_connect
@@
 	(wire
 		(pts
-			(xy 114.3 105.41) (xy 106.68 105.41)
+			(xy 43.18 69.85) (xy 35.56 69.85)
 		)
 		(stroke
@@
 	(wire
 		(pts
-			(xy 114.3 102.87) (xy 106.68 102.87)
+			(xy 43.18 72.39) (xy 35.56 72.39)
 		)
 		(stroke
@@
 	(wire
 		(pts
-			(xy 114.3 97.79) (xy 106.68 97.79)
+			(xy 43.18 77.47) (xy 35.56 77.47)
 		)
 		(stroke
@@
 	(wire
 		(pts
-			(xy 114.3 92.71) (xy 106.68 92.71)
+			(xy 114.3 85.09) (xy 106.68 85.09)
 		)
 		(stroke
@@
 		)
 	)
-	(global_label "CAL_GPIO20"
+	(global_label "CAL_GPIO22"
 		(shape passive)
 		(at 213.36 259.08 180)
@@
 	(global_label "RANGE_CH3"
 		(shape passive)
-		(at 106.68 97.79 180)
-		(effects
-			(font
-				(size 1.016 1.016)
-			)
-			(justify right)
-		)
-		(property "Intersheetrefs" "${INTERSHEET_REFS}"
-			(at 106.68 97.79 0)
+		(at 35.56 77.47 180)
+		(effects
+			(font
+				(size 1.016 1.016)
+			)
+			(justify right)
+		)
+		(property "Intersheetrefs" "${INTERSHEET_REFS}"
+			(at 35.56 77.47 0)
 			(hide yes)
 			(show_name no)
@@
 	(global_label "RANGE_CH2"
 		(shape passive)
-		(at 106.68 102.87 180)
-		(effects
-			(font
-				(size 1.016 1.016)
-			)
-			(justify right)
-		)
-		(property "Intersheetrefs" "${INTERSHEET_REFS}"
-			(at 106.68 102.87 0)
+		(at 35.56 72.39 180)
+		(effects
+			(font
+				(size 1.016 1.016)
+			)
+			(justify right)
+		)
+		(property "Intersheetrefs" "${INTERSHEET_REFS}"
+			(at 35.56 72.39 0)
 			(hide yes)
 			(show_name no)
@@
 	(global_label "RANGE_CH1"
 		(shape passive)
-		(at 106.68 105.41 180)
-		(effects
-			(font
-				(size 1.016 1.016)
-			)
-			(justify right)
-		)
-		(property "Intersheetrefs" "${INTERSHEET_REFS}"
-			(at 106.68 105.41 0)
+		(at 35.56 69.85 180)
+		(effects
+			(font
+				(size 1.016 1.016)
+			)
+			(justify right)
+		)
+		(property "Intersheetrefs" "${INTERSHEET_REFS}"
+			(at 35.56 69.85 0)
 			(hide yes)
 			(show_name no)
@@
 		)
 	)
-	(global_label "CAL_GPIO20"
-		(shape passive)
-		(at 106.68 92.71 180)
-		(effects
-			(font
-				(size 1.016 1.016)
-			)
-			(justify right)
-		)
-		(property "Intersheetrefs" "${INTERSHEET_REFS}"
-			(at 106.68 92.71 0)
-			(hide yes)
-			(show_name no)
+	(global_label "CAL_GPIO22"
+		(shape passive)
+		(at 106.68 85.09 180)
+		(effects
+			(font
+				(size 1.016 1.016)
+			)
+			(justify right)
+		)
+		(property "Intersheetrefs" "${INTERSHEET_REFS}"
+			(at 106.68 85.09 0)
+			(hide yes)
+			(show_name no)
