File: Pico2/hardware/pilyzer-afe/kicad/pilyzer-afe.kicad_sch (KiCad schematic)
At the start: 36 parts, among them J5 Logic D0–D7 + GND, J6 Pico 2 socket, J7 Pico 2 socket, U1 TLV9064IDR, U2 TS5A23159DGSR, U3 TS5A23159DGSR, U4 TLV9064IDR

Commit message: Put logic on GPIO6-13 and the range controls on GPIO2-4 on every board
The PL2407AFE already had them there; the bare Pico 2 and the PiLyzer
AFE had logic on GPIO8-15 and ranges on GPIO4-6. Now D0 is GPIO6 on
every board, as the generator is GPIO16 on every board. GPIO0/1 stay
free for a UART.

- Firmware 1.13 (0x010D).
- PiLyzer AFE schematic: range nets on J6.4-6, D0-D7 on J6.9-17,
  no-connects on J6.1, 2, 7, 19, 20. check_kicad.py passes against it
  and against board_config.h; ERC is clean; the preview is re-exported.
- READMEs updated, including the firmware pin table, which had still
  listed the ranges on 16-18 and the test output on 20.

Co-Authored-By: Claude Opus 5 <noreply@anthropic.com>
Connections:
- net RANGE_CH1: now also J6.4 (Pin_4); no longer J6.6 (Pin_6)
- net RANGE_CH2: now also J6.5 (Pin_5); no longer J6.7 (Pin_7)
- net RANGE_CH3: now also J6.6 (Pin_6); no longer J6.9 (Pin_9)
- net D1_GPIO7: now reaches J6.10 (Pin_10)
- net D1_GPIO7: now also R20.2, R28.1
- net D0_GPIO8 renamed D0_GPIO6
- net D0_GPIO6: now also J6.9 (Pin_9); no longer J6.11 (Pin_11)
- removed net D1_GPIO9: J6.12 (Pin_12), R20.2, R28.1
- net D2_GPIO10 renamed D2_GPIO8
- net D2_GPIO8: now also J6.11 (Pin_11); no longer J6.14 (Pin_14)
- net D3_GPIO11 renamed D3_GPIO9
- net D3_GPIO9: now also J6.12 (Pin_12); no longer J6.15 (Pin_15)
- net D4_GPIO12 renamed D4_GPIO10
- net D4_GPIO10: now also J6.14 (Pin_14); no longer J6.16 (Pin_16)
- net D5_GPIO13 renamed D5_GPIO11
- net D5_GPIO11: now also J6.15 (Pin_15); no longer J6.17 (Pin_17)
- net D6_GPIO14 renamed D6_GPIO12
- net D6_GPIO12: now also J6.16 (Pin_16); no longer J6.19 (Pin_19)
- net D7_GPIO15 renamed D7_GPIO13
- net D7_GPIO13: now also J6.17 (Pin_17); no longer J6.20 (Pin_20)
Other:
- note added: "ADC GPIO26–28; logic GPIO6–13; range GPIO2–4; test GPIO22; generator GPIO16–19."
- note removed: "ADC GPIO26–28; logic GPIO8–15; range GPIO4–6; test GPIO22; generator GPIO16–19."
Changed lines of the file:
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@@
 		)
 	)
-	(text "ADC GPIO26–28; logic GPIO8–15; range GPIO4–6; test GPIO22; generator GPIO16–19."
+	(text "ADC GPIO26–28; logic GPIO6–13; range GPIO2–4; test GPIO22; generator GPIO16–19."
 		(exclude_from_sim no)
 		(at 12.7 142.24 0)
@@
 	)
 	(no_connect
-		(at 43.18 80.01)
-	)
-	(no_connect
 		(at 114.3 97.79)
 	)
@@
 	)
 	(no_connect
-		(at 43.18 64.77)
-	)
-	(no_connect
 		(at 114.3 59.69)
 	)
@@
 	)
 	(no_connect
-		(at 43.18 67.31)
-	)
-	(no_connect
 		(at 114.3 102.87)
 	)
@@
 	(wire
 		(pts
-			(xy 43.18 105.41) (xy 35.56 105.41)
-		)
-		(stroke
-			(width 0.1524)
-			(type default)
-		)
-	)
-	(wire
-		(pts
 			(xy 114.3 62.23) (xy 106.68 62.23)
 		)
@@
 	(wire
 		(pts
-			(xy 43.18 72.39) (xy 35.56 72.39)
-		)
-		(stroke
-			(width 0.1524)
-			(type default)
-		)
-	)
-	(wire
-		(pts
 			(xy 280.67 54.61) (xy 280.67 49.53)
 		)
@@
 	(wire
 		(pts
-			(xy 43.18 102.87) (xy 35.56 102.87)
-		)
-		(stroke
-			(width 0.1524)
-			(type default)
-		)
-	)
-	(wire
-		(pts
 			(xy 346.71 100.33) (xy 351.79 100.33)
 		)
@@
 		)
 	)
-	(global_label "D4_GPIO12"
+	(global_label "D6_GPIO12"
 		(shape passive)
 		(at 35.56 95.25 180)
@@
 		)
 	)
-	(global_label "D6_GPIO14"
+	(global_label "D6_GPIO12"
 		(shape passive)
 		(at 372.11 95.25 180)
@@
 		)
 	)
-	(global_label "D5_GPIO13"
+	(global_label "D7_GPIO13"
 		(shape passive)
 		(at 35.56 97.79 180)
@@
 		)
 	)
-	(global_label "D7_GPIO15"
+	(global_label "D7_GPIO13"
 		(shape passive)
 		(at 372.11 118.11 180)
@@
 		)
 	)
-	(global_label "D7_GPIO15"
-		(shape passive)
-		(at 35.56 105.41 180)
-		(effects
-			(font
-				(size 1.016 1.016)
-			)
-			(justify right)
-		)
-		(property "Intersheetrefs" "${INTERSHEET_REFS}"
-			(at 35.56 105.41 0)
-			(hide yes)
-			(show_name no)
-			(do_not_autoplace no)
-			(effects
-				(font
-					(size 1.016 1.016)
-				)
-			)
-		)
-	)
 	(global_label "GND"
 		(shape passive)
@@
 		)
 	)
-	(global_label "D1_GPIO9"
+	(global_label "D3_GPIO9"
 		(shape passive)
 		(at 35.56 85.09 180)
@@
 		)
 	)
-	(global_label "D4_GPIO12"
+	(global_label "D4_GPIO10"
 		(shape passive)
 		(at 351.79 54.61 0)
@@
 		)
 	)
-	(global_label "D1_GPIO9"
+	(global_label "D1_GPIO7"
 		(shape passive)
 		(at 280.67 72.39 180)
@@
 		)
 	)
-	(global_label "D0_GPIO8"
+	(global_label "D0_GPIO6"
 		(shape passive)
 		(at 280.67 49.53 180)
@@
 		)
 	)
-	(global_label "D2_GPIO10"
+	(global_label "D2_GPIO8"
 		(shape passive)
 		(at 280.67 95.25 180)
@@
 		)
 	)
-	(global_label "D3_GPIO11"
+	(global_label "D5_GPIO11"
 		(shape passive)
 		(at 35.56 92.71 180)
@@
 		)
 	)
-	(global_label "RANGE_CH3"
+	(global_label "D0_GPIO6"
 		(shape passive)
 		(at 35.56 77.47 180)
@@
 		)
 	)
-	(global_label "D4_GPIO12"
+	(global_label "D4_GPIO10"
 		(shape passive)
 		(at 372.11 49.53 180)
@@
 		)
 	)
-	(global_label "RANGE_CH2"
-		(shape passive)
-		(at 35.56 72.39 180)
-		(effects
-			(font
-				(size 1.016 1.016)
-			)
-			(justify right)
-		)
-		(property "Intersheetrefs" "${INTERSHEET_REFS}"
-			(at 35.56 72.39 0)
-			(hide yes)
-			(show_name no)
-			(do_not_autoplace no)
-			(effects
-				(font
-					(size 1.016 1.016)
-				)
-			)
-		)
-	)
 	(global_label "D6_IN"
 		(shape passive)
@@
 		)
 	)
-	(global_label "D0_GPIO8"
+	(global_label "D0_GPIO6"
 		(shape passive)
 		(at 260.35 54.61 0)
@@
 		)
 	)
-	(global_label "D5_GPIO13"
+	(global_label "D5_GPIO11"
 		(shape passive)
 		(at 351.79 77.47 0)
@@
 		)
 	)
-	(global_label "D3_GPIO11"
+	(global_label "D3_GPIO9"
 		(shape passive)
 		(at 280.67 118.11 180)
@@
 		)
 	)
-	(global_label "D2_GPIO10"
+	(global_label "D4_GPIO10"
 		(shape passive)
 		(at 35.56 90.17 180)
@@
 		)
 	)
-	(global_label "RANGE_CH1"
+	(global_label "RANGE_CH3"
 		(shape passive)
 		(at 35.56 69.85 180)
@@
 		)
 	)
-	(global_label "D7_GPIO15"
+	(global_label "D7_GPIO13"
 		(shape passive)
 		(at 351.79 123.19 0)
@@
 		)
 	)
-	(global_label "D3_GPIO11"
+	(global_label "D3_GPIO9"
 		(shape passive)
 		(at 260.35 123.19 0)
@@
 		)
 	)
-	(global_label "D2_GPIO10"
+	(global_label "D2_GPIO8"
 		(shape passive)
 		(at 260.35 100.33 0)
@@
 		)
 	)
-	(global_label "D5_GPIO13"
+	(global_label "D5_GPIO11"
 		(shape passive)
 		(at 372.11 72.39 180)
@@
 		)
 	)
-	(global_label "D6_GPIO14"
-		(shape passive)
-		(at 35.56 102.87 180)
-		(effects
-			(font
-				(size 1.016 1.016)
-			)
-			(justify right)
-		)
-		(property "Intersheetrefs" "${INTERSHEET_REFS}"
-			(at 35.56 102.87 0)
-			(hide yes)
-			(show_name no)
-			(do_not_autoplace no)
-			(effects
-				(font
-					(size 1.016 1.016)
-				)
-			)
-		)
-	)
 	(global_label "+3V3"
 		(shape passive)
@@
 		)
 	)
-	(global_label "D6_GPIO14"
+	(global_label "D6_GPIO12"
 		(shape passive)
 		(at 351.79 100.33 0)
@@
 		)
 	)
-	(global_label "D1_GPIO9"
+	(global_label "D1_GPIO7"
 		(shape passive)
 		(at 260.35 77.47 0)
@@
 		)
 	)
-	(global_label "D0_GPIO8"
+	(global_label "D2_GPIO8"
 		(shape passive)
 		(at 35.56 82.55 180)
@@
 (global_label "GND" (shape passive) (at 320.04 194.31 270) (effects (font (size 1.016 1.016)) (justify right)) (property "Intersheetrefs" "${INTERSHEET_REFS}" (at 320.04 194.31 270) (effects (font (size 1.016 1.016)) (hide yes))))
 (text "U4: anti-alias filters U4A/B/C on the channel sheets; U4D tied off, U4E is the supply unit." (at 250 172.72 0) (effects (font (size 1.016 1.016)) (justify left bottom)))
+	(no_connect
+		(at 43.18 72.39)
+	)
+	(no_connect
+		(at 43.18 102.87)
+	)
+	(no_connect
+		(at 43.18 105.41)
+	)
+	(wire
+		(pts
+			(xy 43.18 64.77) (xy 35.56 64.77)
+		)
+		(stroke
+			(width 0.1524)
+			(type default)
+		)
+	)
+	(global_label "RANGE_CH1"
+		(shape passive)
+		(at 35.56 64.77 180)
+		(effects
+			(font
+				(size 1.016 1.016)
+			)
+			(justify right)
+		)
+		(property "Intersheetrefs" "${INTERSHEET_REFS}"
+			(at 35.56 64.77 0)
+			(hide yes)
+			(show_name no)
+			(do_not_autoplace no)
+			(effects
+				(font
+					(size 1.016 1.016)
+				)
+			)
+		)
+	)
+	(wire
+		(pts
+			(xy 43.18 67.31) (xy 35.56 67.31)
+		)
+		(stroke
+			(width 0.1524)
+			(type default)
+		)
+	)
+	(global_label "RANGE_CH2"
+		(shape passive)
+		(at 35.56 67.31 180)
+		(effects
+			(font
+				(size 1.016 1.016)
+			)
+			(justify right)
+		)
+		(property "Intersheetrefs" "${INTERSHEET_REFS}"
+			(at 35.56 67.31 0)
+			(hide yes)
+			(show_name no)
+			(do_not_autoplace no)
+			(effects
+				(font
+					(size 1.016 1.016)
+				)
+			)
+		)
+	)
+	(wire
+		(pts
+			(xy 43.18 80.01) (xy 35.56 80.01)
+		)
+		(stroke
+			(width 0.1524)
+			(type default)
+		)
+	)
+	(global_label "D1_GPIO7"
+		(shape passive)
+		(at 35.56 80.01 180)
+		(effects
+			(font
+				(size 1.016 1.016)
+			)
+			(justify right)
+		)
+		(property "Intersheetrefs" "${INTERSHEET_REFS}"
+			(at 35.56 80.01 0)
+			(hide yes)
+			(show_name no)
+			(do_not_autoplace no)
+			(effects
+				(font
+					(size 1.016 1.016)
+				)
+			)
+		)
+	)
 	(sheet_instances
 		(path "/"
