File: Pico2/hardware/pilyzer-lite/kicad/pilyzer-lite.kicad_sch (KiCad schematic)
At the start: 32 parts, among them J5 Logic D0–D7 + GND, J6 Pico 2 socket, J7 Pico 2 socket, U1 TLV9064IDR, U4 TLV9064IDR

Commit message: Move the Lite's square wave to GPIO22 as well
The same change as rev A's, minus the range nets: the Lite has no
analogue switch, so only CAL_GPIO20 on J7.15 had to become CAL_GPIO22 on
J7.12, with the no-connect flag swapping to the pad it left. The sheet
note now says the generator has GPIO16-19 rather than that they are
unused.

check_lite.py passes its 25 groups and ERC stays at 0 and 0. Only the
root preview is re-exported; the two channel sheets were unchanged, so
they keep the files they had rather than a new timestamp. These previews
are exported without a background, unlike rev A's — each project keeps
the way its own were made.

Co-Authored-By: Claude Opus 5 <noreply@anthropic.com>
Connections:
- net CAL_GPIO22: now reaches J7.12 (Pin_12)
- net CAL_GPIO22: now also R35.1
- net CAL_GPIO20: no longer names the net of J7.15 (Pin_15)
- net CAL_GPIO20: no longer R35.1
Other:
- note added: "ADC GPIO26–27; logic GPIO8–15; test GPIO22; generator GPIO16–19. GPIO4–6 unused."
- note removed: "Firmware 1.7: ADC GPIO26–27; logic GPIO8–15; test GPIO20. GPIO16–18 unused."
Changed lines of the file:
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@@
 		)
 	)
-	(text "Firmware 1.7: ADC GPIO26–27; logic GPIO8–15; test GPIO20. GPIO16–18 unused."
+	(text "ADC GPIO26–27; logic GPIO8–15; test GPIO22; generator GPIO16–19. GPIO4–6 unused."
 		(exclude_from_sim no)
 		(at 12.7 142.24 0)
@@
 	)
 	(no_connect
-		(at 114.3 85.09)
+		(at 114.3 92.71)
 	)
 	(no_connect
@@
 	(wire
 		(pts
-			(xy 114.3 92.71) (xy 106.68 92.71)
+			(xy 114.3 85.09) (xy 106.68 85.09)
 		)
 		(stroke
@@
 		)
 	)
-	(global_label "CAL_GPIO20"
+	(global_label "CAL_GPIO22"
 		(shape passive)
 		(at 213.36 259.08 180)
@@
 		)
 	)
-	(global_label "CAL_GPIO20"
-		(shape passive)
-		(at 106.68 92.71 180)
-		(effects
-			(font
-				(size 1.016 1.016)
-			)
-			(justify right)
-		)
-		(property "Intersheetrefs" "${INTERSHEET_REFS}"
-			(at 106.68 92.71 0)
-			(hide yes)
-			(show_name no)
+	(global_label "CAL_GPIO22"
+		(shape passive)
+		(at 106.68 85.09 180)
+		(effects
+			(font
+				(size 1.016 1.016)
+			)
+			(justify right)
+		)
+		(property "Intersheetrefs" "${INTERSHEET_REFS}"
+			(at 106.68 85.09 0)
+			(hide yes)
+			(show_name no)
